Commit message: A more robust simulation

File: src/dip_sim/urdf/dip_2.urdf (robot description, URDF)
Before this commit: robot double_pendulum_2, 3 links, 2 joints
Joints:
- joint joint1: limit effort=10 velocity=5 -> effort=1e9 velocity=5
- joint joint2: limit effort=1 velocity=5 -> effort=1e9 velocity=5; origin xyz=0 0.0508 0.0129 rpy=0 0 0 -> xyz=0 0.0508 0 rpy=0 0 0
